Commit message: move baselink to center car_1

File: src/racecar_simulator/racecar0.xacro (robot description, xacro)
@@ -10,5 +10,5 @@
   <xacro:property name="wheel_radius" value="0.0508" />
   <xacro:property name="wheel_length" value="0.0381" />
-  <xacro:property name="laser_distance_from_base_link" value="0.275" />
+  <xacro:property name="laser_distance_from_base_link" value="0.12" />
   <xacro:property name="laser_height" value="0.05" />
   <xacro:property name="laser_radius" value="0.026" />
@@ -21,5 +21,5 @@
   <link name="base_link$(arg prefix)">
     <visual>
-      <origin xyz="${wheelbase/2} 0 ${ground_offset+height/2}"/>
+      <origin xyz="0 0 ${ground_offset+height/2}"/>
       <geometry>
         <box size="${wheelbase} ${width} ${height}"/>
@@ -44,5 +44,5 @@
     <parent link="base_link$(arg prefix)"/>
     <child link="back_left_wheel$(arg prefix)"/>
-    <origin xyz="0 ${(wheel_length+width)/2} ${wheel_radius}"/>
+    <origin xyz="${-wheelbase/2} ${(wheel_length+width)/2} ${wheel_radius}"/>
   </joint>
   <link name="back_left_wheel$(arg prefix)">
@@ -58,5 +58,5 @@
     <parent link="base_link$(arg prefix)"/>
     <child link="back_right_wheel$(arg prefix)"/>
-    <origin xyz="0 ${-(wheel_length+width)/2} ${wheel_radius}"/>
+    <origin xyz="${-wheelbase/2} ${-(wheel_length+width)/2} ${wheel_radius}"/>
   </joint>
   <link name="back_right_wheel$(arg prefix)">
@@ -72,5 +72,5 @@
     <parent link="base_link$(arg prefix)"/>
     <child link="front_left_hinge$(arg prefix)"/>
-    <origin xyz="${wheelbase} ${(wheel_length+width)/2} ${wheel_radius}"/>
+    <origin xyz="${wheelbase/2} ${(wheel_length+width)/2} ${wheel_radius}"/>
   </joint>
   <link name="front_left_hinge$(arg prefix)"/>
@@ -91,5 +91,5 @@
     <parent link="base_link$(arg prefix)"/>
     <child link="front_right_hinge$(arg prefix)"/>
-    <origin xyz="${wheelbase} ${-(wheel_length+width)/2} ${wheel_radius}"/>
+    <origin xyz="${wheelbase/2} ${-(wheel_length+width)/2} ${wheel_radius}"/>
   </joint>
   <link name="front_right_hinge$(arg prefix)"/>
