Commit message: foxy version

File: src/racecar_simulator/params/racecar0.xacro (robot description, xacro)
@@ -19,5 +19,5 @@
     <color rgba="0.3 0.57 1. 1."/>
   </material>
-  <link name="base_link$(arg prefix)">
+  <link name="base_link">
     <visual>
       <origin xyz="0 0 ${ground_offset+height/2}"/>
@@ -28,10 +28,10 @@
     </visual>
   </link>
-  <joint name="base_to_laser_model$(arg prefix)" type="fixed">
-    <parent link="base_link$(arg prefix)"/>
-    <child link="laser_model$(arg prefix)"/>
+  <joint name="base_to_laser" type="fixed">
+    <parent link="base_link"/>
+    <child link="laser"/>
     <origin xyz="${laser_distance_from_base_link} 0 ${ground_offset+height+(laser_height/2)}"/>
   </joint>
-  <link name="laser_model$(arg prefix)">
+  <link name="laser">
     <visual>
       <geometry>
@@ -41,10 +41,10 @@
     </visual>
   </link>
-  <joint name="base_to_back_left_wheel$(arg prefix)" type="fixed">
-    <parent link="base_link$(arg prefix)"/>
-    <child link="back_left_wheel$(arg prefix)"/>
+  <joint name="base_to_back_left_wheel" type="fixed">
+    <parent link="base_link"/>
+    <child link="back_left_wheel"/>
     <origin xyz="${-wheelbase/2} ${(wheel_length+width)/2} ${wheel_radius}"/>
   </joint>
-  <link name="back_left_wheel$(arg prefix)">
+  <link name="back_left_wheel">
     <visual>
       <geometry>
@@ -55,10 +55,10 @@
     </visual>
   </link>
-  <joint name="base_to_back_right_wheel$(arg prefix)" type="fixed">
-    <parent link="base_link$(arg prefix)"/>
-    <child link="back_right_wheel$(arg prefix)"/>
+  <joint name="base_to_back_right_wheel" type="fixed">
+    <parent link="base_link"/>
+    <child link="back_right_wheel"/>
     <origin xyz="${-wheelbase/2} ${-(wheel_length+width)/2} ${wheel_radius}"/>
   </joint>
-  <link name="back_right_wheel$(arg prefix)">
+  <link name="back_right_wheel">
     <visual>
       <geometry>
@@ -69,15 +69,15 @@
     </visual>
   </link>
-  <joint name="base_to_front_left_hinge$(arg prefix)" type="fixed">
-    <parent link="base_link$(arg prefix)"/>
-    <child link="front_left_hinge$(arg prefix)"/>
+  <joint name="base_to_front_left_hinge" type="fixed">
+    <parent link="base_link"/>
+    <child link="front_left_hinge"/>
     <origin xyz="${wheelbase/2} ${(wheel_length+width)/2} ${wheel_radius}"/>
   </joint>
-  <link name="front_left_hinge$(arg prefix)"/>
-  <joint name="front_left_hinge_to_wheel$(arg prefix)" type="continuous">
-    <parent link="front_left_hinge$(arg prefix)"/>
-    <child link="front_left_wheel$(arg prefix)"/>
+  <link name="front_left_hinge"/>
+  <joint name="front_left_hinge_to_wheel" type="continuous">
+    <parent link="front_left_hinge"/>
+    <child link="front_left_wheel"/>
   </joint>
-  <link name="front_left_wheel$(arg prefix)">
+  <link name="front_left_wheel">
     <visual>
       <geometry>
@@ -88,15 +88,15 @@
     </visual>
   </link>
-  <joint name="base_to_front_right_hinge$(arg prefix)" type="fixed">
-    <parent link="base_link$(arg prefix)"/>
-    <child link="front_right_hinge$(arg prefix)"/>
+  <joint name="base_to_front_right_hinge" type="fixed">
+    <parent link="base_link"/>
+    <child link="front_right_hinge"/>
     <origin xyz="${wheelbase/2} ${-(wheel_length+width)/2} ${wheel_radius}"/>
   </joint>
-  <link name="front_right_hinge$(arg prefix)"/>
-  <joint name="front_right_hinge_to_wheel$(arg prefix)" type="continuous">
-    <parent link="front_right_hinge$(arg prefix)"/>
-    <child link="front_right_wheel$(arg prefix)"/>
+  <link name="front_right_hinge"/>
+  <joint name="front_right_hinge_to_wheel" type="continuous">
+    <parent link="front_right_hinge"/>
+    <child link="front_right_wheel"/>
   </joint>
-  <link name="front_right_wheel$(arg prefix)">
+  <link name="front_right_wheel">
     <visual>
       <geometry>
